File: CPU_Flex_AGB/CPU_Flex_AGB.kicad_pcb (KiCad board)
At the start: 2 copper layers, 17.4 x 15.9 mm, 5 parts, among them J1 Conn_01x16, J2 CPU_AGB_A_Interface

Commit message: Updated PCBs
Parts:
- moved B+ 2.75 mm to (177.5, 92.6), turned to 180 degrees
- moved G 2.75 mm to (180.3, 92.6), turned to 180 degrees
Routing:
- net VCC: track 24.1 -> 21.3 mm
- net Net-(J2-Pad2): track 6.67 -> 6.59 mm, vias 2 -> 1
Other:
- board text added: "v20220310"
- board text removed: "v20220202"
