File: shield/GBAHD_Shield.kicad_sch (KiCad schematic)
At the start: 43 parts, among them J1 Conn_01x01, J10 Conn_01x10, J11 Conn_02x03_Odd_Even, J2 FFC_OGBA_32, J3 FFC_GBA-SP, J4 Conn_01x16, J5 FFC_OGBA_40, J6 Conn_01x06, J7 Conn_01x08, J8 Conn_01x10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

Commit message: Updated PCBs
Parts:
- added C4: 47uF, Capacitor_SMD:C_0805_2012Metric_Pad1.18x1.45mm_HandSolder, symbol Device:C
Connections:
- net GND: now also C4.1
- net VCC: now also C4.2
Other:
- moved on the sheet: JP1
Changed lines of the file:
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@@
   (title_block
     (title "gbaHD Shield")
-    (date "2022-02-28")
+    (date "2022-03-10")
     (rev "v2")
     (comment 1 "made by: ManCloud")
-    (comment 2 "Version: v20220228")
+    (comment 2 "Version: v20220310")
   )
   (junction (at 138.43 40.64) (diameter 0) (color 0 0 0 0)
@@
     (stroke (width 0) (type default) (color 0 0 0 0))
   )
-  (wire (pts (xy 69.85 102.87) (xy 69.85 99.06))
+  (wire (pts (xy 64.77 105.41) (xy 64.77 101.6))
     (stroke (width 0) (type default) (color 0 0 0 0))
   )
@@
     (stroke (width 0) (type default) (color 0 0 0 0))
   )
-  (wire (pts (xy 54.61 102.87) (xy 54.61 99.06))
+  (wire (pts (xy 49.53 105.41) (xy 49.53 101.6))
     (stroke (width 0) (type default) (color 0 0 0 0))
   )
@@
     (stroke (width 0) (type default) (color 0 0 0 0))
   )
-  (wire (pts (xy 62.23 99.06) (xy 62.23 97.79))
+  (wire (pts (xy 57.15 101.6) (xy 57.15 100.33))
     (stroke (width 0) (type default) (color 0 0 0 0))
   )
@@
     (stroke (width 0) (type default) (color 0 0 0 0))
   )
+  (wire (pts (xy 71.12 106.68) (xy 71.12 107.95))
+    (stroke (width 0) (type default) (color 0 0 0 0))
+  )
   (wire (pts (xy 208.28 143.51) (xy 207.01 143.51))
     (stroke (width 0) (type default) (color 0 0 0 0))
@@
     (stroke (width 0) (type default) (color 0 0 0 0))
   )
-  (wire (pts (xy 57.15 102.87) (xy 54.61 102.87))
+  (wire (pts (xy 52.07 105.41) (xy 49.53 105.41))
     (stroke (width 0) (type default) (color 0 0 0 0))
   )
@@
     (stroke (width 0) (type default) (color 0 0 0 0))
   )
+  (wire (pts (xy 71.12 97.79) (xy 71.12 99.06))
+    (stroke (width 0) (type default) (color 0 0 0 0))
+  )
   (wire (pts (xy 262.89 78.74) (xy 261.62 78.74))
     (stroke (width 0) (type default) (color 0 0 0 0))
@@
     (stroke (width 0) (type default) (color 0 0 0 0))
   )
-  (wire (pts (xy 67.31 102.87) (xy 69.85 102.87))
+  (wire (pts (xy 62.23 105.41) (xy 64.77 105.41))
     (stroke (width 0) (type default) (color 0 0 0 0))
   )
@@
     (pin "1")
   )
-  (symbol (lib_id "Jumper:SolderJumper_3_Open") (at 62.23 102.87 180) (unit 1)
+  (symbol (lib_id "Jumper:SolderJumper_3_Open") (at 57.15 105.41 180) (unit 1)
     (in_bom yes) (on_board yes)
-    (property "Reference" "JP1" (id 0) (at 62.23 105.7402 0))
-    (property "Value" "SolderJumper_3_Open" (id 1) (at 62.23 108.0516 0))
-    (property "Footprint" "Jumper:SolderJumper-3_P1.3mm_Open_Pad1.0x1.5mm_NumberLabels" (id 2) (at 62.23 102.87 0)
+    (property "Reference" "JP1" (id 0) (at 57.15 108.2802 0))
+    (property "Value" "SolderJumper_3_Open" (id 1) (at 57.15 110.5916 0))
+    (property "Footprint" "Jumper:SolderJumper-3_P1.3mm_Open_Pad1.0x1.5mm_NumberLabels" (id 2) (at 57.15 105.41 0)
       (effects (font (size 1.27 1.27)) hide)
     )
-    (property "Datasheet" "~" (id 3) (at 62.23 102.87 0)
+    (property "Datasheet" "~" (id 3) (at 57.15 105.41 0)
       (effects (font (size 1.27 1.27)) hide)
     )
@@
     (pin "3")
   )
-  (symbol (lib_id "power:+4V") (at 54.61 99.06 0) (unit 1)
+  (symbol (lib_id "power:+4V") (at 49.53 101.6 0) (unit 1)
     (in_bom yes) (on_board yes)
-    (property "Reference" "#PWR010" (id 0) (at 54.61 102.87 0)
+    (property "Reference" "#PWR010" (id 0) (at 49.53 105.41 0)
       (effects (font (size 1.27 1.27)) hide)
     )
-    (property "Value" "+4V" (id 1) (at 54.991 94.6658 0))
-    (property "Footprint" "" (id 2) (at 54.61 99.06 0)
+    (property "Value" "+4V" (id 1) (at 49.911 97.2058 0))
+    (property "Footprint" "" (id 2) (at 49.53 101.6 0)
       (effects (font (size 1.27 1.27)) hide)
     )
-    (property "Datasheet" "" (id 3) (at 54.61 99.06 0)
+    (property "Datasheet" "" (id 3) (at 49.53 101.6 0)
       (effects (font (size 1.27 1.27)) hide)
     )
@@
     (pin "1")
   )
-  (symbol (lib_id "power:+3V3") (at 69.85 99.06 0) (unit 1)
+  (symbol (lib_id "power:+3V3") (at 64.77 101.6 0) (unit 1)
     (in_bom yes) (on_board yes)
-    (property "Reference" "#PWR012" (id 0) (at 69.85 102.87 0)
+    (property "Reference" "#PWR012" (id 0) (at 64.77 105.41 0)
       (effects (font (size 1.27 1.27)) hide)
     )
-    (property "Value" "+3V3" (id 1) (at 70.231 94.6658 0))
-    (property "Footprint" "" (id 2) (at 69.85 99.06 0)
+    (property "Value" "+3V3" (id 1) (at 65.151 97.2058 0))
+    (property "Footprint" "" (id 2) (at 64.77 101.6 0)
       (effects (font (size 1.27 1.27)) hide)
     )
-    (property "Datasheet" "" (id 3) (at 69.85 99.06 0)
+    (property "Datasheet" "" (id 3) (at 64.77 101.6 0)
       (effects (font (size 1.27 1.27)) hide)
     )
@@
     (pin "1")
   )
-  (symbol (lib_id "power:VCC") (at 62.23 97.79 0) (unit 1)
+  (symbol (lib_id "power:VCC") (at 57.15 100.33 0) (unit 1)
     (in_bom yes) (on_board yes)
-    (property "Reference" "#PWR0104" (id 0) (at 62.23 101.6 0)
+    (property "Reference" "#PWR0104" (id 0) (at 57.15 104.14 0)
       (effects (font (size 1.27 1.27)) hide)
     )
-    (property "Value" "VCC" (id 1) (at 62.611 93.3958 0))
-    (property "Footprint" "" (id 2) (at 62.23 97.79 0)
+    (property "Value" "VCC" (id 1) (at 57.531 95.9358 0))
+    (property "Footprint" "" (id 2) (at 57.15 100.33 0)
       (effects (font (size 1.27 1.27)) hide)
     )
-    (property "Datasheet" "" (id 3) (at 62.23 97.79 0)
+    (property "Datasheet" "" (id 3) (at 57.15 100.33 0)
       (effects (font (size 1.27 1.27)) hide)
     )
@@
     (pin "2")
   )
+  (symbol (lib_id "Device:C") (at 71.12 102.87 180) (unit 1)
+    (in_bom yes) (on_board yes)
+    (property "Reference" "C4" (id 0) (at 69.85 100.33 0))
+    (property "Value" "47uF" (id 1) (at 73.66 105.41 0))
+    (property "Footprint" "Capacitor_SMD:C_0805_2012Metric_Pad1.18x1.45mm_HandSolder" (id 2) (at 70.1548 99.06 0)
+      (effects (font (size 1.27 1.27)) hide)
+    )
+    (property "Datasheet" "~" (id 3) (at 71.12 102.87 0)
+      (effects (font (size 1.27 1.27)) hide)
+    )
+    (pin "1")
+    (pin "2")
+  )
+  (symbol (lib_id "power:GND") (at 71.12 107.95 0) (unit 1)
+    (in_bom yes) (on_board yes)
+    (property "Reference" "#PWR0101" (id 0) (at 71.12 114.3 0)
+      (effects (font (size 1.27 1.27)) hide)
+    )
+    (property "Value" "GND" (id 1) (at 71.247 112.3442 0))
+    (property "Footprint" "" (id 2) (at 71.12 107.95 0)
+      (effects (font (size 1.27 1.27)) hide)
+    )
+    (property "Datasheet" "" (id 3) (at 71.12 107.95 0)
+      (effects (font (size 1.27 1.27)) hide)
+    )
+    (pin "1")
+  )
+  (symbol (lib_id "power:VCC") (at 71.12 97.79 0) (unit 1)
+    (in_bom yes) (on_board yes)
+    (property "Reference" "#PWR0116" (id 0) (at 71.12 101.6 0)
+      (effects (font (size 1.27 1.27)) hide)
+    )
+    (property "Value" "VCC" (id 1) (at 71.501 93.3958 0))
+    (property "Footprint" "" (id 2) (at 71.12 97.79 0)
+      (effects (font (size 1.27 1.27)) hide)
+    )
+    (property "Datasheet" "" (id 3) (at 71.12 97.79 0)
+      (effects (font (size 1.27 1.27)) hide)
+    )
+    (pin "1")
+  )
   (sheet_instances
     (path "/" (page "1"))
@@
       (reference "#PWR041") (unit 1) (value "GND") (footprint "")
     )
+    (path "/65ca5973-f0ba-492d-ba0c-29098cd4af01"
+      (reference "#PWR0101") (unit 1) (value "GND") (footprint "")
+    )
     (path "/00000000-0000-0000-0000-0000608c1a96"
       (reference "#PWR0102") (unit 1) (value "GND") (footprint "")
@@
       (reference "#PWR0115") (unit 1) (value "+3V3") (footprint "")
     )
+    (path "/c5ec9dc4-3568-4fed-a55f-f0a55aff7482"
+      (reference "#PWR0116") (unit 1) (value "VCC") (footprint "")
+    )
     (path "/00000000-0000-0000-0000-0000608bc7c6"
       (reference "C1") (unit 1) (value "100nF") (footprint "Capacitor_SMD:C_0805_2012Metric_Pad1.18x1.45mm_HandSolder")
@@
       (reference "C3") (unit 1) (value "100nF") (footprint "Capacitor_SMD:C_0805_2012Metric_Pad1.18x1.45mm_HandSolder")
     )
+    (path "/352c5f65-5f4a-4cde-bd04-648895f9a231"
+      (reference "C4") (unit 1) (value "47uF") (footprint "Capacitor_SMD:C_0805_2012Metric_Pad1.18x1.45mm_HandSolder")
+    )
     (path "/00000000-0000-0000-0000-000061842569"
