File: breakout_OGBA/GBABreakout.kicad_pcb (KiCad board)
At the start: 2 copper layers, 19.9 x 10 mm, 19 parts, among them J1 Conn_01x16, J10 TP8, J11 TP3, J12 TP2, J13 S02, J14 S01, J15 OSC, J16 EX1, J17 G, J2 VCC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

Commit message: Develop (#16)
* Remove get_components from Makefile, fix bluepad path

* Fixed naming of submodule

* Fixed submodule mess

* Removed bluepad32

* Re-Add Bluepad32 properly

* Update Build for adding web/bitstream handler

* Add implementation for web handler and bitstream handler

* Update arduino version

* Fix build by using bluepad template as component foundation

* Removed bluepad submodule

* Copying default component files

* Remove get_components

* Improved over all build config

* Overall refactoring and added wifi and mega handler

* Minor updates to sdkconfig

* Add first crude version to update firmware

* Remove Bluepad Debug outputs

* some cleanup

* updated .gitignore and added some files

* updated gitmodules

* fixed submodules

* Update Upgrade function

* Fix gitignore

* Fix SPIFFS upload

* a little bit of tinkering

* Changed order of run/init to be faster for TWI

* Removed endTransmission after requestFrom

* changed twi handling

* added definition for bigger I2C-Buffer

* some cleanup

* remove wifi

* Fix sending of inputs without controller available

* Fix WiFi

* fixed button mapping

* fixed button mappings and polling intervalls

* Improve Timer Code

* Refactoring and Preferences

* Add Prefs

* Add prefs

* fixed verify_flash() --> missing beginTransmission()

* Added Bluetooth Mapping, Preferences Refactoring

* Add bluetooth cfg

* Refactoring

* Remove template

* CMake fixes

* changed TWI handling - added data validity timeout

* some cleanup

* Added License Hadder

* updated CPU-flex

* Refactoring

* Beautifying

* Update Bitstream

* refactored avr-firmware to be makefile project

* added controller detection

* Better layout

* Better shield handling

* Better OTA

* For now - only load bitstream from SPIFFS to be faster

* Add Force option for ATMega update

* Added Force Option for Mega Update

* Upd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
Other:
- net class Default removed
- net class PWR removed
